Commit message: bugfix: tilt sensor rays with their mount

File: flatsim/tests/testbot.urdf (robot description, URDF)
Before this commit: robot testbot, 6 links, 5 joints
Links:
- added link camera_link
Joints:
- added joint camera_joint: type fixed, parent base_link, child camera_link, origin xyz=0.25 0 0.4 rpy=0 -0.2576 0
